File: FETProbe_tiny.kicad_pcb (KiCad board)
At the start: 2 copper layers, 23 x 15 mm, 17 parts, among them J1 u.Fl, J5 u.Fl, Q1 BF998

Commit message: updated gerbers and assembly info
Changed lines of the file:
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@@
     (aux_axis_origin 100 100)
     (pcbplotparams
-      (layerselection 0x0020000_7ffffffe)
+      (layerselection 0x00010fc_ffffffff)
       (disableapertmacros false)
-      (usegerberextensions false)
+      (usegerberextensions true)
       (usegerberattributes true)
-      (usegerberadvancedattributes true)
-      (creategerberjobfile true)
+      (usegerberadvancedattributes false)
+      (creategerberjobfile false)
       (svguseinch false)
       (svgprecision 6)
-      (excludeedgelayer false)
+      (excludeedgelayer true)
       (plotframeref false)
       (viasonmask false)
@@
       (psa4output false)
       (plotreference true)
-      (plotvalue true)
+      (plotvalue false)
       (plotinvisibletext false)
       (sketchpadsonfab false)
-      (subtractmaskfromsilk false)
-      (outputformat 2)
+      (subtractmaskfromsilk true)
+      (outputformat 1)
       (mirror false)
       (drillshape 0)
-      (scaleselection 4)
-      (outputdirectory "")
+      (scaleselection 1)
+      (outputdirectory "gerbers/")
     )
   )
@@
     (fp_line (start 1.6 -0.8) (end -1.2 -0.8) (layer "F.Fab") (width 0.1))
     (fp_line (start -1.2 -0.8) (end -1.6 -0.4) (layer "F.Fab") (width 0.1))
-    (pad "1" smd roundrect (at -1.35 0 180) (size 1.4 1.35) (layers "F.Cu" "F.Paste" "F.Mask") (roundrect_rratio 0.185185)
+    (pad "1" smd roundrect (at -1.35 0 180) (size 1.4 1.35) (layers "F.Cu" "F.Paste" "F.Mask") (roundrect_rratio 0.1851851852)
       (net 9 "+5V") (pintype "passive"))
-    (pad "2" smd roundrect (at 1.35 0 180) (size 1.4 1.35) (layers "F.Cu" "F.Paste" "F.Mask") (roundrect_rratio 0.185185)
+    (pad "2" smd roundrect (at 1.35 0 180) (size 1.4 1.35) (layers "F.Cu" "F.Paste" "F.Mask") (roundrect_rratio 0.1851851852)
       (net 1 "GND") (pintype "passive"))
     (model "${KICAD6_3DMODEL_DIR}/Capacitor_Tantalum_SMD.3dshapes/CP_EIA-3216-18_Kemet-A.wrl"
@@
     (fp_line (start 1.6 0.8) (end -1.6 0.8) (layer "F.Fab") (width 0.1))
     (fp_line (start -1.6 -0.8) (end 1.6 -0.8) (layer "F.Fab") (width 0.1))
-    (pad "1" smd roundrect (at -1.475 0) (size 1.15 1.8) (layers "F.Cu" "F.Paste" "F.Mask") (roundrect_rratio 0.217391)
+    (pad "1" smd roundrect (at -1.475 0) (size 1.15 1.8) (layers "F.Cu" "F.Paste" "F.Mask") (roundrect_rratio 0.2173913043)
       (net 4 "/out2") (pintype "passive"))
-    (pad "2" smd roundrect (at 1.475 0) (size 1.15 1.8) (layers "F.Cu" "F.Paste" "F.Mask") (roundrect_rratio 0.217391)
+    (pad "2" smd roundrect (at 1.475 0) (size 1.15 1.8) (layers "F.Cu" "F.Paste" "F.Mask") (roundrect_rratio 0.2173913043)
       (net 5 "/out1") (pintype "passive"))
     (model "${KICAD6_3DMODEL_DIR}/Capacitor_SMD.3dshapes/C_1206_3216Metric.wrl"

Commit message: minor: update component properties in layout
Parts:
- C3: value 10uF -> 100uF
Changed lines of the file:
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@@
       (effects (font (size 0.5 0.5) (thickness 0.06)))
     )
-    (fp_text value "10uF" (at 0 -0.4) (layer "F.Fab")
+    (fp_text value "100uF" (at 0 -0.4) (layer "F.Fab")
       (effects (font (size 0.5 0.5) (thickness 0.06)))
     )
@@
     (property "Sheetfile" "FETProbe_tiny.kicad_sch")
     (property "Sheetname" "")
-    (attr exclude_from_pos_files)
+    (property "exclude_from_bom" "")
+    (attr exclude_from_pos_files exclude_from_bom)
     (fp_text reference "C4" (at 0.33 1.06 unlocked) (layer "F.SilkS") hide
       (effects (font (size 0.5 0.5) (thickness 0.06)))
