File: FETProbe_tiny.kicad_sch (KiCad schematic)
At the start: 17 parts, among them J1 u.Fl, J5 u.Fl, Q1 BF998

Commit message: updated gerbers and assembly info
Parts:
- C1: value 10uF -> (none); footprint Capacitor_SMD:C_0402_1005Metric -> (none); voltage (none) -> 10V
- C3: value 10uF -> (none); footprint Capacitor_Tantalum_SMD:CP_EIA-3216-18_Kemet-A -> (none); voltage (none) -> 6V3
- C4: value C -> (none); footprint FETProbe:input_cap -> (none); now left out of the parts list
- C5: value 100nF -> (none); footprint Capacitor_SMD:C_1206_3216Metric -> (none); dielectric (none) -> NP0
- C6, C7: value 2.2pF -> (none); footprint Capacitor_SMD:C_0402_1005Metric -> (none); dielectric (none) -> NP0
- D2: value RB531SM-30FH -> (none); footprint Diode_SMD:D_SOD-523 -> (none); comment (none) -> just about any schottky will do
- J1, J5: value u.Fl -> (none); footprint Connector_Coaxial:U.FL_Molex_MCRF_73412-0110_Vertical -> (none)
- L1: value 10nH -> (none); footprint Inductor_SMD:L_0402_1005Metric -> (none)
- N1: comment (none) -> remove one sidewall
- Q1: value BF998 -> (none); footprint FETProbe:SOT-143_mod -> (none)
- R1: value 4k7 -> (none); footprint Resistor_SMD:R_0402_1005Metric -> (none); comment (none) -> general purpose; dielectric (none) -> 1%
- R2: value 6k8 -> (none); footprint Resistor_SMD:R_0402_1005Metric -> (none); comment (none) -> general purpose; dielectric (none) -> 1%
- R3: value 1M -> (none); footprint Resistor_SMD:R_0402_1005Metric -> (none); comment (none) -> general purpose; dielectric (none) -> 1%
- R4: value 47R -> (none); footprint Resistor_SMD:R_0402_1005Metric -> (none); comment (none) -> general purpose; dielectric (none) -> 1%
- TP3: value TestPoint -> (none); footprint TestPoint:TestPoint_THTPad_D2.0mm_Drill1.0mm -> (none)

Commit message: Add LCSC numbers
Parts:
- C1: value (none) -> 10uF; footprint (none) -> Capacitor_SMD:C_0402_1005Metric; LCSC (none) -> C15525
- C3: value (none) -> 100uF; footprint (none) -> Capacitor_Tantalum_SMD:CP_EIA-3216-18_Kemet-A; LCSC (none) -> C122251
- C4: value (none) -> C; footprint (none) -> FETProbe:input_cap
- C5: value (none) -> 100nF; footprint (none) -> Capacitor_SMD:C_1206_3216Metric; LCSC (none) -> C97946
- C6, C7: value (none) -> 2.2pF; footprint (none) -> Capacitor_SMD:C_0402_1005Metric; LCSC (none) -> C437438
- D2: value (none) -> RB531SM-30FH; footprint (none) -> Diode_SMD:D_SOD-523; LCSC (none) -> C50676
- J1, J5: value (none) -> u.Fl; footprint (none) -> Connector_Coaxial:U.FL_Molex_MCRF_73412-0110_Vertical; LCSC (none) -> C88374
- L1: value (none) -> 10nH; footprint (none) -> Inductor_SMD:L_0402_1005Metric; LCSC (none) -> C382409
- N1: value (none) -> Laird_BMI-S-101; footprint (none) -> RF_Shielding:Laird_Technologies_BMI-S-101_13.66x12.70mm
- Q1: value (none) -> BF998; footprint (none) -> FETProbe:SOT-143_mod; LCSC (none) -> C108141
- R1: value (none) -> 4k7; footprint (none) -> Resistor_SMD:R_0402_1005Metric; LCSC (none) -> C25900
- R2: value (none) -> 6k8; footprint (none) -> Resistor_SMD:R_0402_1005Metric; LCSC (none) -> C25917
- R3: value (none) -> 1M; footprint (none) -> Resistor_SMD:R_0402_1005Metric; LCSC (none) -> C26083
- R4: value (none) -> 47R; footprint (none) -> Resistor_SMD:R_0402_1005Metric; LCSC (none) -> C25118
- TP3: value (none) -> TestPoint; footprint (none) -> TestPoint:TestPoint_THTPad_D2.0mm_Drill1.0mm; now left out of the parts list
